Commit message: 改变雷达放置位置

File: src/unitree_guide/unitree_ros/robots/a1_description/xacro/robot.xacro (robot description, xacro)
@@ -128,5 +128,5 @@
     <!-- 对于连接 -->
     <joint name="laser_livox_joint" type="fixed" >
-        <origin xyz="0.0 0 0.1" rpy="0 0.785 0" />
+        <origin xyz="0.0 0 0.08" rpy="0 0 0" />
         <parent link="base" />
         <child link="laser_livox"/>

Commit message: 修改了发布点云坐标系关系，现在的点云是正确的

File: src/unitree_guide/unitree_ros/robots/a1_description/xacro/robot.xacro (robot description, xacro)
@@ -128,5 +128,5 @@
     <!-- 对于连接 -->
     <joint name="laser_livox_joint" type="fixed" >
-        <origin xyz="0.0 0 0.08" rpy="0 0 0" />
+        <origin xyz="0.2 0 0.08" rpy="0 0.785 0" />
         <parent link="base" />
         <child link="laser_livox"/>
